File: circuit/Finishline Display.sch (EAGLE design)
At the start: 25 parts, among them U1 PCA9501, U2 HEF4066BT, U3 TM1637

Commit message: changes circuit to include capacitors
This change adds resistors and capacitors to the LED driver chip
as well as individual caps to each WS2812 LED.
Parts:
- removed S1: SWS004, smd-special:SWS004
- added C1, C2: 1nF, rcl:C-EUC0805
- added C10, C11, C4, C5, C6, C7, C8, C9: 100nF, rcl:C-EUC0805
- added C3: 10nF, rcl:C-EUC0805
- added R10, R9: 10K, resistor:R-EU_M0805
- added SW1: 416131160804, Wurth_Elektronik_Electromechanic_Switchs_rev15b:416131160804
Connections:
- net +5V: now also C10.2, C11.2, C5.2, C6.2, C7.2, C8.2, C9.2
- net 0V: now also C1.1, C10.1, C11.1, C2.1, C3.2, C4.2, C5.1, C6.1, C7.1, C8.1, C9.1, SW1.1, SW1.2, SW1.3, SW1.4; no longer S1.1, S1.2, S1.3, S1.4
- net 3.3V: now also C3.1, C4.1, R10.2, R9.2
- net N$14: now also SW1.8; no longer S1.8
- net N$15: now also SW1.7; no longer S1.7
- net N$16: now also SW1.6; no longer S1.6
- net N$17: now also SW1.5; no longer S1.5
- net N$18: now also C1.2, R9.1
- net N$19: now also C2.2, R10.1

Commit message: add Controller brd+sch, fix Display LDR line
An additional board for the controller was added as a Due shield.
The LDR was hooked up to a digital pin, has been changed to use
a separate line which gets patched through the 4066.
Parts:
- removed C1, C2: 1nF, rcl:C-EUC0805
- removed C10, C11, C4, C5, C6, C7, C8, C9: 100nF, rcl:C-EUC0805
- removed C3: 10nF, rcl:C-EUC0805
- removed R10, R9: 10K, resistor:R-EU_M0805
- removed SW1: 416131160804, Wurth_Elektronik_Electromechanic_Switchs_rev15b:416131160804
- added S1: SWS004, smd-special:SWS004
- JP1, JP2: device pinhead:PINHD-1X8 -> pinhead:PINHD-1X9
Connections:
- removed net 0V: C1.1, C10.1, C11.1, C2.1, C3.2, C4.2, C5.1, C6.1, C7.1, C8.1, C9.1, JP1.8, JP2.8, LED1.GND, LED2.GND, LED3.GND, LED4.GND, LED5.GND, LED6.GND, LED7.GND, R8.2, SW1.1, SW1.2, SW1.3, SW1.4, U1.A4, U1.A5, U1.GND, U1._WC, U2.3E, U2.4E, U2.VSS, U3.GND
- new net GND: JP1.9, JP2.9, LED1.GND, LED2.GND, LED3.GND, LED4.GND, LED5.GND, LED6.GND, LED7.GND, R8.2, S1.1, S1.2, S1.3, S1.4, U1.A4, U1.A5, U1.GND, U1._WC, U2.4E, U2.VSS, U3.GND
- new net LDR: JP1.8, JP2.8, U2.3Y
- new net N$23: U1.IO2, U2.3E
- net +5V: no longer C10.2, C11.2, C5.2, C6.2, C7.2, C8.2, C9.2
- net 3.3V: no longer C3.1, C4.1, R10.2, R9.2
- net N$14: now also S1.8; no longer SW1.8
- net N$15: now also S1.7; no longer SW1.7
- net N$16: now also S1.6; no longer SW1.6
- net N$17: now also S1.5; no longer SW1.5
- net N$18: no longer C1.2, R9.1
- net N$19: no longer C2.2, R10.1
- net N$20: now also U2.3Z; no longer U1.IO2
Other:
- note added: "+5V +3.3V WS2812DATA SCL SDA CLK DIO LDR GND"
- moved on the sheet: R7, R8

Commit message: finalize display module and controller shield
Display Module: Reordered the WS2813 LEDs to be consistent with normal
7-segment LED numbers (a-g). Changed schematics to be in the same
orientation as the board in top view. Re-adds the capacitors for the
WS2812 LEDs and the LDR line, which inadvertently got lost in the last
commit. Added silk screen.

Controller Shield: Added large electrolyte capacitor to buffer for the
WS2812 LEDs. Added a series resistor for the WS2812 data line. Added
silk screen and corrected wrong pinout of the I2C and serial header.
Parts:
- removed S1: SWS004, smd-special:SWS004
- added C1, C2: 1nF, rcl:C-EUC0805
- added C10, C11, C4, C5, C6, C7, C8, C9: 100nF, rcl:C-EUC0805
- added C3: 10nF, rcl:C-EUC0805
- added R10, R9: 10K, resistor:R-EU_M0805
- added SW1: 416131160804, Wurth_Elektronik_Electromechanic_Switchs_rev15b:416131160804
Connections:
- removed net 3.3V: JP1.2, JP2.2, R1.2, R2.2, R3.2, R4.2, R5.1, R6.1, R7.2, U1.3.3V, U2.VDD, U3.3.3V
- new net +3V3: C3.1, C4.1, JP1.2, JP2.2, R1.2, R10.2, R2.2, R3.2, R4.2, R5.1, R6.1, R7.2, R9.2, U1.3.3V, U2.VDD, U3.3.3V
- net +5V: now also C10.1, C11.1, C5.1, C6.1, C7.1, C8.1, C9.1
- net GND: now also C1.1, C10.2, C11.2, C2.1, C3.2, C4.2, C5.2, C6.2, C7.2, C8.2, C9.2, SW1.1, SW1.2, SW1.3, SW1.4; no longer S1.1, S1.2, S1.3, S1.4
- net N$14: now also SW1.8; no longer S1.8
- net N$15: now also SW1.7; no longer S1.7
- net N$16: now also SW1.6; no longer S1.6
- net N$17: now also SW1.5; no longer S1.5
- net N$18: now also C1.2, R9.1
- net N$19: now also C2.2, R10.1
Other:
- note removed: "+5V +3.3V WS2812DATA SCL SDA CLK DIO LDR GND"
- moved on the sheet: JP1, JP2, R1, R2, R3, R4, R7, R8, U1
