File: circuit/Startgate Controller-Motherboard.sch (EAGLE design)
At the start: 25 parts, among them IC1 MAX3490ESA, IC2 L293D, U2 HEF4066BT, U3 HEF4066BT, U4 HEF4066BT, U5 HEF4066BT, X1 RJ45-8L21-B, X2 SOLENOID

Commit message: correct some schematics mistakes and add gerber files
A demo mode button was added to the controller, the layout of the
controller shield as well as the startgate displays were changed.
Parts:
- removed JP3, JP4: (no value), pinhead:PINHD-1X13
- removed U$1: TCA9548A, miro:TCA9548A
- removed U$2, U$3, U$4, U$5: RFID-RC522, miro:RFID-RC522
- removed U$6, U$7, U$8, U$9: DISPLAY-OLED-128X32, diy-modules:DISPLAY-OLED-128X32
- removed U3, U4, U5: HEF4066BT, NXP_By_element14_Batch_1:HEF4066BT
- JP1: value (none) -> LEFT
- JP2: value (none) -> RIGHT
- JP5: value (none) -> FTDI
- R1, R2: value (none) -> 120
- U1: value (none) -> PROMINI
- U2: value HEF4066BT -> TCA9548A; device NXP_By_element14_Batch_1:HEF4066BT -> miro:TCA9548A
Connections:
- removed net MISO-OUT1: U$2.MISO, U2.4Z
- removed net MISO-OUT2: U$3.MISO, U3.4Z
- removed net MISO-OUT3: U$4.MISO, U4.4Z
- removed net MISO-OUT4: U$5.MISO, U5.4Z
- removed net MOSI-OUT1: U$2.MOSI, U2.3Z
- removed net MOSI-OUT2: U$3.MOSI, U3.3Z
- removed net MOSI-OUT3: U$4.MOSI, U4.3Z
- removed net MOSI-OUT4: U$5.MOSI, U5.3Z
- removed net N$13: IC2.GND1, IC2.GND2, IC2.GND3, IC2.GND4, X1.2, X1.8, X2-2.KL
- removed net SCK-OUT1: U$2.SCK, U2.2Z
- removed net SCK-OUT2: U$3.SCK, U3.2Z
- removed net SCK-OUT3: U$4.SCK, U4.2Z
- removed net SCK-OUT4: U$5.SCK, U5.2Z
- removed net SS-OUT1: U$2.SDA, U2.1Z
- removed net SS-OUT2: U$3.SDA, U3.1Z
- removed net SS-OUT3: U$4.SDA, U4.1Z
- removed net SS-OUT4: U$5.SDA, U5.1Z
- net +12V: now also IC2.VCC2
- net +3V3: now also U2.+3V3; no longer JP3.1, JP4.1, U$1.+3V3, U$2.+3V3, U$3.+3V3, U$4.+3V3, U$5.+3V3, U$6.VCC, U$7.VCC, U$8.VCC, U$9.VCC, U2.VDD, U3.VDD, U4.VDD, U5.VDD
- net +5V: now also IC2.1-2EN
- net ENA1: no longer JP3.2, U2.1E, U2.2E, U2.3E, U2.4E
- net ENA2: no longer JP3.12, U3.1E, U3.2E, U3.3E, U3.4E
- net ENA3: no longer JP4.2, U4.1E, U4.2E, U4.3E, U4.4E
- net ENA4: no longer JP4.12, U5.1E, U5.2E, U5.3E, U5.4E
- net GND: now also IC2.2A, IC2.3-4EN, IC2.3A, IC2.4A, IC2.GND1, IC2.GND2, IC2.GND3, IC2.GND4, U2.A0, U2.A1, U2.A2, U2.GND, X1.2, X1.8, X2-2.KL; no longer JP3.13, JP4.13, U$1.A0, U$1.A1, U$1.A2, U$1.GND, U$2.GND, U$3.GND, U$4.GND, U$5.GND, U$6.GND, U$7.GND, U$8.GND, U$9.GND, U2.VSS, U3.VSS, U4.VSS, U5.VSS
- net MISO: no longer JP3.7, JP4.7, U2.4Y, U3.4Y, U4.4Y, U5.4Y
- net MOSI: no longer JP3.6, JP4.6, U2.3Y, U3.3Y, U4.3Y, U5.3Y
- net N$5: now also U2.SCL; no longer U$1.SCL
- net N$6: now also U2.SDA; no longer U$1.SDA
- net RST: no longer JP3.9, JP4.9, U$2.RST, U$3.RST, U$4.RST, U$5.RST
- net SCK: no longer JP3.8, JP4.8, U2.2Y, U3.2Y, U4.2Y, U5.2Y
- net SCL1: now also U2.SC2; no longer JP3.4, U$1.SC2, U$6.SCL
- net SCL2: now also U2.SC3; no longer JP3.10, U$1.SC3, U$7.SCL
- net SCL3: now also U2.SC6; no longer JP4.4, U$1.SC6, U$8.SCL
- net SCL4: now also U2.SC7; no longer JP4.10, U$1.SC7, U$9.SCL
- net SDA1: now also U2.SD2; no longer JP3.3, U$1.SD2, U$6.SDA
- net SDA2: now also U2.SD3; no longer JP3.11, U$1.SD3, U$7.SDA
- net SDA3: now also U2.SD6; no longer JP4.3, U$1.SD6, U$8.SDA
- net SDA4: now also U2.SD7; no longer JP4.11, U$1.SD7, U$9.SDA
- net SS: no longer JP3.5, JP4.5, U2.1Y, U3.1Y, U4.1Y, U5.1Y
Other:
- moved on the sheet: IC1, IC2, JP1, JP2, JP5, R1, R2, U1, X1, X2-1, X2-2
