File: circuit/Finishline Controller.sch (EAGLE design)
At the start: 23 parts, among them IC1 74HCT245N, IC2 MAX3490ESA

Commit message: create the final schematics and boards
Some schematics errors have been corrected. Another connector for
the laser diodes of the Finishing Gate has been added. The
connectors to the daughterboards have been rotated, so that the
cabling will run mostly straight.

All gerber files have been added as well as .zip files for the
boardhouse.
Parts:
- added JP6: lASER, pinhead:PINHD-1X2
- POWER: value 8x1F-H8.5 -> POWER; device SmartPrj:PINHD-1X8 -> pinhead:PINHD-1X7
Connections:
- net +3V3: now also POWER.1, POWER.3; no longer POWER.2, POWER.4
- net +5V: now also POWER.4; no longer POWER.5
- net GND: now also JP6.2, POWER.5; no longer POWER.7
- net MASTER-RESET: now also POWER.2; no longer POWER.3
- net PIN32: now also JP6.1
- net RX2: now also JP3.2; no longer JP3.1
- net TX2: now also JP3.1; no longer JP3.2
- net VIN: now also POWER.7; no longer POWER.8
Other:
- moved on the sheet: JP2, JP3, R4
Changed lines of the file:
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@@
 <clearance class="4" value="0.6096"/>
+</class>
+<class number="5" name="12V" width="0.3048" drill="0.4064">
+<clearance class="5" value="0.6096"/>
 </class>
 </classes>
@@
 <part name="GND5" library="supply1" deviceset="GND" device=""/>
 <part name="+5V" library="supply1" deviceset="+5V" device=""/>
-<part name="POWER" library="SmartPrj" deviceset="PINHD-1X8" device="" value="8x1F-H8.5"/>
+<part name="POWER" library="pinhead" deviceset="PINHD-1X7" device="" value="POWER"/>
 <part name="ADCL" library="SmartPrj" deviceset="PINHD-1X8" device="" value="8x1F-H8.5"/>
 <part name="COMMUNICATION" library="SmartPrj" deviceset="PINHD-1X8" device="" value="8x1F-H8.5"/>
@@
 <part name="GND1" library="supply1" deviceset="GND" device=""/>
 <part name="JP3" library="pinhead" deviceset="PINHD-1X3" device="" value="RASPI"/>
+<part name="JP6" library="pinhead" deviceset="PINHD-1X2" device="" value="lASER"/>
+<part name="GND2" library="supply1" deviceset="GND" device=""/>
 </parts>
 <sheets>
@@
 <instance part="12V" gate="-2" x="469.9" y="251.46"/>
 <instance part="C1" gate="G$1" x="314.96" y="218.44"/>
-<instance part="R4" gate="G$1" x="180.34" y="243.84" rot="R90"/>
-<instance part="JP2" gate="G$1" x="190.5" y="220.98"/>
-<instance part="GND1" gate="1" x="180.34" y="210.82"/>
-<instance part="JP3" gate="A" x="314.96" y="177.8"/>
+<instance part="R4" gate="G$1" x="314.96" y="180.34" rot="R90"/>
+<instance part="JP2" gate="G$1" x="325.12" y="157.48"/>
+<instance part="GND1" gate="1" x="314.96" y="147.32"/>
+<instance part="JP3" gate="A" x="292.1" y="160.02"/>
+<instance part="JP6" gate="G$1" x="383.54" y="157.48"/>
+<instance part="GND2" gate="1" x="370.84" y="147.32"/>
 </instances>
 <busses>
@@
 <wire x1="474.98" y1="320.04" x2="474.98" y2="335.28" width="0.1524" layer="91"/>
 <pinref part="+5V" gate="1" pin="+5V"/>
-<pinref part="POWER" gate="A" pin="5"/>
+<pinref part="POWER" gate="A" pin="4"/>
 <label x="472.44" y="340.36" size="1.778" layer="95"/>
 </segment>
@@
 <wire x1="474.98" y1="314.96" x2="474.98" y2="309.88" width="0.1524" layer="91"/>
 <junction x="490.22" y="314.96"/>
-<pinref part="POWER" gate="A" pin="7"/>
 <pinref part="POWER" gate="A" pin="6"/>
+<pinref part="POWER" gate="A" pin="5"/>
 <pinref part="GND5" gate="1" pin="GND"/>
 </segment>
@@
 <pinref part="GND1" gate="1" pin="GND"/>
 <pinref part="JP2" gate="G$1" pin="2"/>
-<wire x1="180.34" y1="213.36" x2="180.34" y2="220.98" width="0.1524" layer="91"/>
-<wire x1="180.34" y1="220.98" x2="187.96" y2="220.98" width="0.1524" layer="91"/>
+<wire x1="314.96" y1="149.86" x2="314.96" y2="157.48" width="0.1524" layer="91"/>
+<wire x1="314.96" y1="157.48" x2="322.58" y2="157.48" width="0.1524" layer="91"/>
 </segment>
 <segment>
 <pinref part="JP3" gate="A" pin="3"/>
-<wire x1="312.42" y1="175.26" x2="287.02" y2="175.26" width="0.1524" layer="91"/>
-<label x="294.64" y="175.26" size="1.778" layer="95"/>
+<wire x1="289.56" y1="157.48" x2="264.16" y2="157.48" width="0.1524" layer="91"/>
+<label x="271.78" y="157.48" size="1.778" layer="95"/>
+</segment>
+<segment>
+<pinref part="JP6" gate="G$1" pin="2"/>
+<pinref part="GND2" gate="1" pin="GND"/>
+<wire x1="381" y1="157.48" x2="370.84" y2="157.48" width="0.1524" layer="91"/>
+<wire x1="370.84" y1="157.48" x2="370.84" y2="149.86" width="0.1524" layer="91"/>
 </segment>
 </net>
@@
 <wire x1="495.3" y1="312.42" x2="480.06" y2="312.42" width="0.1524" layer="91"/>
 <label x="480.06" y="312.42" size="1.778" layer="95"/>
-<pinref part="POWER" gate="A" pin="8"/>
+<pinref part="POWER" gate="A" pin="7"/>
 </segment>
 </net>
@@
 <pinref part="XIO" gate="A" pin="13"/>
 </segment>
+<segment>
+<pinref part="JP6" gate="G$1" pin="1"/>
+<wire x1="381" y1="160.02" x2="355.6" y2="160.02" width="0.1524" layer="91"/>
+<label x="363.22" y="160.02" size="1.778" layer="95"/>
+</segment>
 </net>
 <net name="PIN34" class="0">
@@
 </segment>
 <segment>
-<pinref part="JP3" gate="A" pin="1"/>
-<wire x1="312.42" y1="180.34" x2="287.02" y2="180.34" width="0.1524" layer="91"/>
-<label x="294.64" y="180.34" size="1.778" layer="95"/>
+<pinref part="JP3" gate="A" pin="2"/>
+<wire x1="289.56" y1="160.02" x2="264.16" y2="160.02" width="0.1524" layer="91"/>
+<label x="271.78" y="160.02" size="1.778" layer="95"/>
 </segment>
 </net>
@@
 </segment>
 <segment>
-<pinref part="JP3" gate="A" pin="2"/>
-<wire x1="312.42" y1="177.8" x2="287.02" y2="177.8" width="0.1524" layer="91"/>
-<label x="294.64" y="177.8" size="1.778" layer="95"/>
+<pinref part="JP3" gate="A" pin="1"/>
+<wire x1="289.56" y1="162.56" x2="264.16" y2="162.56" width="0.1524" layer="91"/>
+<label x="271.78" y="162.56" size="1.778" layer="95"/>
 </segment>
 </net>
@@
 <segment>
 <label x="462.28" y="325.12" size="1.778" layer="95"/>
-<pinref part="POWER" gate="A" pin="3"/>
+<pinref part="POWER" gate="A" pin="2"/>
 <wire x1="495.3" y1="325.12" x2="462.28" y2="325.12" width="0.1524" layer="91"/>
 </segment>
@@
 <segment>
 <pinref part="R4" gate="G$1" pin="1"/>
-<wire x1="180.34" y1="238.76" x2="180.34" y2="233.68" width="0.1524" layer="91"/>
+<wire x1="314.96" y1="175.26" x2="314.96" y2="170.18" width="0.1524" layer="91"/>
 <pinref part="JP2" gate="G$1" pin="1"/>
-<wire x1="180.34" y1="233.68" x2="180.34" y2="223.52" width="0.1524" layer="91"/>
-<wire x1="187.96" y1="223.52" x2="180.34" y2="223.52" width="0.1524" layer="91"/>
-<wire x1="180.34" y1="233.68" x2="203.2" y2="233.68" width="0.1524" layer="91"/>
-<junction x="180.34" y="233.68"/>
-<label x="190.5" y="233.68" size="1.778" layer="95"/>
+<wire x1="314.96" y1="170.18" x2="314.96" y2="160.02" width="0.1524" layer="91"/>
+<wire x1="322.58" y1="160.02" x2="314.96" y2="160.02" width="0.1524" layer="91"/>
+<wire x1="314.96" y1="170.18" x2="337.82" y2="170.18" width="0.1524" layer="91"/>
+<junction x="314.96" y="170.18"/>
+<label x="325.12" y="170.18" size="1.778" layer="95"/>
 </segment>
 </net>
@@
 </segment>
 </net>
-<net name="+12VEXT" class="0">
+<net name="+12VEXT" class="5">
 <segment>
 <pinref part="RS485" gate="G$1" pin="1"/>
@@
 <segment>
 <pinref part="R4" gate="G$1" pin="2"/>
-<wire x1="180.34" y1="248.92" x2="180.34" y2="259.08" width="0.1524" layer="91"/>
-<label x="180.34" y="251.46" size="1.778" layer="95" rot="R90"/>
+<wire x1="314.96" y1="185.42" x2="314.96" y2="195.58" width="0.1524" layer="91"/>
+<label x="314.96" y="187.96" size="1.778" layer="95" rot="R90"/>
 </segment>
 <segment>
@@
 <junction x="485.14" y="322.58"/>
 <pinref part="+3V3" gate="G$1" pin="+3V3"/>
-<pinref part="POWER" gate="A" pin="4"/>
-<pinref part="POWER" gate="A" pin="2"/>
+<pinref part="POWER" gate="A" pin="3"/>
+<pinref part="POWER" gate="A" pin="1"/>
 <label x="477.52" y="340.36" size="1.778" layer="95"/>
 </segment>
